File: kicad/pulse_v3.sch (KiCad schematic (older format))
At the start: 17 parts, among them P1 12V, P2 LED, P3 ISP, P4 POT, P5 PWM, Q1 BS270, U1 ATTINY45-20PU, U2 LP2950-50LPRE3

Commit message: added alternate part numbers from RS components to schematic and BoM
Parts:
- D1: RS (none) -> BZX79-C4V7,113
- D3: RS (none) -> 1N5819RL
- Q1: RS (none) -> BS170RLRAG
- U1: value ATTINY45-20PU -> ATTINY85-20PU
- U2: RS (none) -> LP2950-50LPRE3
Changed lines of the file:
@@
 P 8050 2925
 F 0 "U1" H 7450 3275 50  0000 L BNN
-F 1 "ATTINY45-20PU" H 7450 3200 50  0000 L BNN
+F 1 "ATTINY85-20PU" H 7450 3200 50  0000 L BNN
 F 2 "DIP-8__300" H 8550 2500 50  0001 C CNN
 F 3 "" H 8050 2925 60  0001 C CNN
@@
 F 2 "TO-92-LDO_LP2950" H 5150 2025 40  0001 C CNN
 F 3 "" H 5150 2025 40  0000 C CNN
+F 4 "LP2950-50LPRE3" H 4950 2350 40  0001 L BNN "RS"
 	1    5150 2025
 	1    0    0    -1
@@
 F 1 "Z4V7" V 7150 3650 40  0000 L BNN
 F 2 "diode_do35_vert" H 7000 3625 60  0001 C CNN
-F 3 "1N5230BTR" H 7000 3525 40  0000 C CNN
+F 3 "1N5230BTR" H 7000 3525 40  0001 C CNN
+F 4 "BZX79-C4V7,113" H 6750 3500 40  0000 L BNN "RS"
 	1    7000 3625
 	0    -1   -1   0
@@
 F 2 "Housings_TO-92:TO-92-FET-molded-wide-universal-DGS" H 10400 3000 60  0001 C CNN
 F 3 "" H 10825 2900 40  0000 C CNN
+F 4 "BS170RLRAG" H 10625 2900 40  0000 L BNN "RS"
 	1    10400 3000
 	1    0    0    -1
@@
 F 2 "diode_do35_vert" H 3450 1975 60  0001 C CNN
 F 3 "" H 3450 1975 60  0000 C CNN
+F 4 "1N5819RL" H 3525 1900 40  0000 L BNN "RS"
 	1    3450 1975
 	1    0    0    -1

Commit message: some part values modified
Parts:
- C1, C2: footprint Capacitor4MMDisc -> pulse:Capacitor4MMDisc
- C3: footprint Capacitor6MMDisc -> pulse:Capacitor6MMDisc
- C4: value 100n -> 1u X7R; footprint Capacitor4MMDisc -> pulse:Capacitor4MMDisc
- D1, D3: footprint diode_do35_vert -> pulse:diode_do35_vert
- P1: footprint Header_12V -> pulse:Header_12V
- P2, P4, P5: footprint pin_strip_3 -> pulse:pin_strip_3
- P3: footprint pin_strip_6b -> pulse:pin_strip_6b
- PB3: footprint Pad01 -> pulse:Pad01
- Q1: footprint Housings_TO-92:TO-92-FET-molded-wide-universal-DGS -> pulse:TO-92-FET-molded-wide-universal-DGS
- R1, R3: footprint res_vert -> pulse:res_vert
- U1: footprint DIP-8__300 -> pulse:DIP-8__300
- U2: footprint TO-92-LDO_LP2950 -> pulse:TO-92-LDO_LP2950
Changed lines of the file:
@@
 F 0 "PB3" V 6625 2550 40  0000 L CNN
 F 1 "ADC3" H 6550 2630 30  0001 C CNN
-F 2 "Pad01" H 6550 2730 30  0001 C CNN
+F 2 "pulse:Pad01" H 6550 2730 30  0001 C CNN
 F 3 "" H 6550 2575 60  0001 C CNN
 	1    6550 2575
@@
 F 0 "P1" V 1550 2075 40  0000 C CNN
 F 1 "12V" V 1650 2075 40  0000 C CNN
-F 2 "Header_12V" V 1750 2075 40  0001 C CNN
+F 2 "pulse:Header_12V" V 1750 2075 40  0001 C CNN
 F 3 "" H 1600 2075 60  0001 C CNN
 	1    1600 2075
@@
 F 0 "U1" H 7450 3275 50  0000 L BNN
 F 1 "ATTINY85-20PU" H 7450 3200 50  0000 L BNN
-F 2 "DIP-8__300" H 8550 2500 50  0001 C CNN
+F 2 "pulse:DIP-8__300" H 8550 2500 50  0001 C CNN
 F 3 "" H 8050 2925 60  0001 C CNN
 	1    8050 2925
@@
 F 0 "P3" V 1550 5050 60  0000 C CNN
 F 1 "ISP" V 1650 5050 60  0000 C CNN
-F 2 "pin_strip_6b" H 1600 5050 60  0001 C CNN
+F 2 "pulse:pin_strip_6b" H 1600 5050 60  0001 C CNN
 F 3 "" H 1600 5050 60  0001 C CNN
 	1    1600 5050
@@
 F 0 "P2" V 1550 1100 40  0000 C CNN
 F 1 "LED" V 1650 1100 40  0000 C CNN
-F 2 "pin_strip_3" H 1600 1100 40  0001 C CNN
+F 2 "pulse:pin_strip_3" H 1600 1100 40  0001 C CNN
 F 3 "" H 1600 1100 40  0000 C CNN
 	1    1600 1100
@@
 F 0 "U2" H 4950 2275 40  0000 L BNN
 F 1 "LP2950-50LPRE3" H 4950 2200 40  0000 L BNN
-F 2 "TO-92-LDO_LP2950" H 5150 2025 40  0001 C CNN
+F 2 "pulse:TO-92-LDO_LP2950" H 5150 2025 40  0001 C CNN
 F 3 "" H 5150 2025 40  0000 C CNN
 F 4 "LP2950-50LPRE3" H 4950 2350 40  0001 L BNN "RS"
@@
 F 0 "D1" V 7200 3650 40  0000 L BNN
 F 1 "Z4V7" V 7150 3650 40  0000 L BNN
-F 2 "diode_do35_vert" H 7000 3625 60  0001 C CNN
+F 2 "pulse:diode_do35_vert" H 7000 3625 60  0001 C CNN
 F 3 "1N5230BTR" H 7000 3525 40  0001 C CNN
 F 4 "BZX79-C4V7,113" H 6750 3500 40  0000 L BNN "RS"
@@
 F 0 "C1" H 6525 3800 40  0000 L BNN
 F 1 "10n" H 6525 3725 40  0000 L BNN
-F 2 "Capacitor4MMDisc" H 6675 3650 60  0001 C CNN
+F 2 "pulse:Capacitor4MMDisc" H 6675 3650 60  0001 C CNN
 F 3 "" H 6675 3650 60  0000 C CNN
 	1    6675 3625
@@
 F 0 "C2" H 8875 3800 40  0000 L CNN
 F 1 "100n" H 8875 3750 40  0000 L CNN
-F 2 "Capacitor4MMDisc" H 9050 3650 60  0001 C CNN
+F 2 "pulse:Capacitor4MMDisc" H 9050 3650 60  0001 C CNN
 F 3 "" H 9050 3650 60  0000 C CNN
 	1    9050 3625
@@
 F 0 "Q1" H 10625 3050 40  0000 L BNN
 F 1 "BS270" H 10625 2975 40  0000 L BNN
-F 2 "Housings_TO-92:TO-92-FET-molded-wide-universal-DGS" H 10400 3000 60  0001 C CNN
+F 2 "pulse:TO-92-FET-molded-wide-universal-DGS" H 10400 3000 60  0001 C CNN
 F 3 "" H 10825 2900 40  0000 C CNN
 F 4 "BS170RLRAG" H 10625 2900 40  0000 L BNN "RS"
@@
 F 0 "R3" V 9855 3075 40  0000 C CNN
 F 1 "2k2" V 9775 3075 40  0000 C CNN
-F 2 "res_vert" H 9775 3075 60  0001 C CNN
+F 2 "pulse:res_vert" H 9775 3075 60  0001 C CNN
 F 3 "" H 9775 3075 60  0000 C CNN
 	1    9775 3075
@@
 F 0 "R1" V 5555 2975 40  0000 C CNN
 F 1 "4k7" V 5475 2975 40  0000 C CNN
-F 2 "res_vert" H 5475 2975 60  0001 C CNN
+F 2 "pulse:res_vert" H 5475 2975 60  0001 C CNN
 F 3 "" H 5475 2975 60  0000 C CNN
 	1    5475 2975
@@
 P 5800 2325
 F 0 "C4" H 5850 2500 40  0000 L BNN
-F 1 "100n" H 5850 2425 40  0000 L BNN
-F 2 "Capacitor4MMDisc" H 5800 2350 60  0001 C CNN
+F 1 "1u X7R" H 5850 2425 40  0000 L BNN
+F 2 "pulse:Capacitor4MMDisc" H 5800 2350 60  0001 C CNN
 F 3 "" H 5800 2350 60  0000 C CNN
 	1    5800 2325
@@
 F 0 "C3" H 4525 2500 40  0000 L BNN
 F 1 "4u7" H 4525 2425 40  0000 L BNN
-F 2 "Capacitor6MMDisc" H 4500 2350 60  0001 C CNN
+F 2 "pulse:Capacitor6MMDisc" H 4500 2350 60  0001 C CNN
 F 3 "" H 4500 2350 60  0000 C CNN
 	1    4500 2325
@@
 F 0 "D3" H 3550 2075 40  0000 L CNN
 F 1 "SB040-E3/54" H 3550 2025 40  0000 L CNN
-F 2 "diode_do35_vert" H 3450 1975 60  0001 C CNN
+F 2 "pulse:diode_do35_vert" H 3450 1975 60  0001 C CNN
 F 3 "" H 3450 1975 60  0000 C CNN
 F 4 "1N5819RL" H 3525 1900 40  0000 L BNN "RS"
@@
 F 0 "P4" V 1550 3300 40  0000 C CNN
 F 1 "POT" V 1650 3300 40  0000 C CNN
-F 2 "pin_strip_3" H 1600 3300 40  0001 C CNN
+F 2 "pulse:pin_strip_3" H 1600 3300 40  0001 C CNN
 F 3 "" H 1600 3300 40  0000 C CNN
 	1    1600 3300
@@
 F 0 "P5" V 1550 4150 40  0000 C CNN
 F 1 "PWM" V 1650 4150 40  0000 C CNN
-F 2 "pin_strip_3" H 1600 4150 40  0001 C CNN
+F 2 "pulse:pin_strip_3" H 1600 4150 40  0001 C CNN
 F 3 "" H 1600 4150 40  0000 C CNN
 	1    1600 4150
